Commit message: Add files via upload

File: src/gantry/urdf/gantry.urdf (robot description, URDF)
Before this commit: robot gantry, 13 links, 12 joints
Links:
- link bs_link: geometry collision mesh filename=package://gantry/meshes/gantry/bs_link.STL; visual mesh filename=package://gantry/meshes/gantry/bs_link.STL
- link linear_rail: geometry collision mesh filename=package://gantry/meshes/gantry/linear_rail.STL; visual mesh filename=package://gantry/meshes/gantry/linear_rail.STL
- link ur_base_link_inertia: geometry collision mesh filename=package://gantry/meshes/ur5e/collision/base.stl; visual mesh filename=package://gantry/meshes/ur5e/visual/base.dae
- link ur_forearm_link: geometry collision mesh filename=package://gantry/meshes/ur5e/collision/forearm.stl; visual mesh filename=package://gantry/meshes/ur5e/visual/forearm.dae
- link ur_shoulder_link: geometry collision mesh filename=package://gantry/meshes/ur5e/collision/shoulder.stl; visual mesh filename=package://gantry/meshes/ur5e/visual/shoulder.dae
- link ur_upper_arm_link: geometry collision mesh filename=package://gantry/meshes/ur5e/collision/upperarm.stl; visual mesh filename=package://gantry/meshes/ur5e/visual/upperarm.dae
- link ur_wrist_1_link: geometry collision mesh filename=package://gantry/meshes/ur5e/collision/wrist1.stl; visual mesh filename=package://gantry/meshes/ur5e/visual/wrist1.dae
- link ur_wrist_2_link: geometry collision mesh filename=package://gantry/meshes/ur5e/collision/wrist2.stl; visual mesh filename=package://gantry/meshes/ur5e/visual/wrist2.dae
- link ur_wrist_3_link: geometry collision mesh filename=package://gantry/meshes/ur5e/collision/wrist3.stl; visual mesh filename=package://gantry/meshes/ur5e/visual/wrist3.dae

Commit message: Add files via upload

File: src/gantry/urdf/gantry.urdf (robot description, URDF)
Before this commit: robot gantry, 13 links, 12 joints
Joints:
- removed joint ur_base_link-base_link_inertia
- added joint base: type fixed, parent ur_base_link, child bs_link, origin xyz=0 0 0 rpy=0 0 0.0, axis 0 0 0
- joint linear_rail_to_ur_base: child ur_base_link -> ur_base_link_inertia
