Commit message: complete cleanup

File: config/curobo/self_collision/ur5e_x.urdf (robot description, URDF)
Before this commit: robot ur5e_robot, 12 links, 11 joints
Links:
- removed link base_link_x
- added link world
Joints:
- removed joint base_fixed
- added joint base_link-base_link_inertia: type fixed, parent base_link, child base_link_inertia, origin xyz=0 0 0 rpy=0 0 3.141592653589793
- joint base_x: child base_link_x -> base_link; limit lower=-1.0 upper=1.0 effort=87 velocity=1.0 -> lower=-10.0 upper=10.0 effort=1000.0 velocity=1.0; origin xyz=0 0 0.0 rpy=0 0 0.0 -> xyz=0 0 0 rpy=0 0 0; parent base_link -> world
